File: FOC.kicad_pcb (KiCad board)
At the start: 0 parts

Commit message: 123
Parts:
- added C1: 100u, Capacitor_Tantalum_SMD:CP_EIA-7343-30_AVX-N_Pad2.25x2.55mm_HandSolder, F.Cu at (116.3, 73.3)
- added C10: 100n, Capacitor_SMD:C_0603_1608Metric_Pad1.08x0.95mm_HandSolder, F.Cu at (135.6, 100.6)
- added C11: 100n, Capacitor_SMD:C_0603_1608Metric_Pad1.08x0.95mm_HandSolder, F.Cu at (140.0, 98.1)
- added C12: 100n, Capacitor_SMD:C_0603_1608Metric_Pad1.08x0.95mm_HandSolder, F.Cu at (135.6, 98.1)
- added C13: 100n, Capacitor_SMD:C_0603_1608Metric_Pad1.08x0.95mm_HandSolder, F.Cu at (140.0, 100.6)
- added C14: 100n, Capacitor_SMD:C_0603_1608Metric_Pad1.08x0.95mm_HandSolder, F.Cu at (135.6, 103.1)
- added C15: 22n, Capacitor_SMD:C_0603_1608Metric_Pad1.08x0.95mm_HandSolder, F.Cu at (134.1, 89.9)
- added C16: 2.2u, Capacitor_SMD:C_0603_1608Metric_Pad1.08x0.95mm_HandSolder, F.Cu at (121.9, 90.4)
- added C17: 1u, Capacitor_SMD:C_0603_1608Metric_Pad1.08x0.95mm_HandSolder, F.Cu at (126.3, 90.4)
- added C18: 1u, Capacitor_SMD:C_0603_1608Metric_Pad1.08x0.95mm_HandSolder, F.Cu at (126.3, 87.9)
- added C19: 22n, Capacitor_SMD:C_0603_1608Metric_Pad1.08x0.95mm_HandSolder, F.Cu at (165.1, 90.4)
- added C2: 15n, Capacitor_SMD:C_0603_1608Metric_Pad1.08x0.95mm_HandSolder, F.Cu at (124.0, 79.8)
- added C20: 4.7u, Capacitor_SMD:C_0603_1608Metric_Pad1.08x0.95mm_HandSolder, F.Cu at (161.0, 73.0)
- added C21: 100n, Capacitor_SMD:C_0603_1608Metric_Pad1.08x0.95mm_HandSolder, F.Cu at (177.0, 69.6)
- added C22: 4.7u, Capacitor_SMD:C_0603_1608Metric_Pad1.08x0.95mm_HandSolder, F.Cu at (181.4, 72.1)
- added C23: 100n, Capacitor_SMD:C_0603_1608Metric_Pad1.08x0.95mm_HandSolder, F.Cu at (177.0, 72.1)
- added C24: 2.2u, Capacitor_SMD:C_0603_1608Metric_Pad1.08x0.95mm_HandSolder, F.Cu at (169.7, 65.5)
- added C25: 1u, Capacitor_SMD:C_0603_1608Metric_Pad1.08x0.95mm_HandSolder, F.Cu at (181.4, 69.6)
- added C26: 1u, Capacitor_SMD:C_0603_1608Metric_Pad1.08x0.95mm_HandSolder, F.Cu at (161.0, 70.5)
- added C27: 15n, Capacitor_SMD:C_0603_1608Metric_Pad1.08x0.95mm_HandSolder, F.Cu at (179.3, 91.9)
- added C3: 100n, Capacitor_SMD:C_0603_1608Metric_Pad1.08x0.95mm_HandSolder, F.Cu at (134.1, 69.6)
- added C4: 47u, Capacitor_Tantalum_SMD:CP_EIA-7343-30_AVX-N_Pad2.25x2.55mm_HandSolder, F.Cu at (132.0, 65.4)
- added C5: 100n, Capacitor_SMD:C_0603_1608Metric_Pad1.08x0.95mm_HandSolder, F.Cu at (139.3, 63.7)
- added C6: 4.7u, Capacitor_SMD:C_0603_1608Metric_Pad1.08x0.95mm_HandSolder, F.Cu at (148.8, 72.1)
- added C7: 100n, Capacitor_SMD:C_0603_1608Metric_Pad1.08x0.95mm_HandSolder, F.Cu at (148.8, 69.6)
- added C8: 4.7u, Capacitor_SMD:C_0603_1608Metric_Pad1.08x0.95mm_HandSolder, F.Cu at (144.5, 72.1)
- added C9: 100n, Capacitor_SMD:C_0603_1608Metric_Pad1.08x0.95mm_HandSolder, F.Cu at (144.5, 69.6)
- added D1: D_S, Diode_SMD:D_SOD-323_HandSoldering, F.Cu at (129.4, 69.8)
- added J1: PWR, Connector_AMASS:AMASS_XT60-M_1x02_P7.20mm_Vertical, F.Cu at (106.2, 69.6)
- added L1: 22u, Inductor_SMD:L_Sumida_CDMC6D28_7.25x6.5mm, F.Cu at (120.4, 61.5)
- added Q1: BSC061N08NS5, Package_TO_SOT_SMD:TDSON-8-1, B.Cu at (116.4, 119.2)
- added Q2: BSC061N08NS5, Package_TO_SOT_SMD:TDSON-8-1, B.Cu at (124.7, 112.5)
- added Q3: BSC061N08NS5, Package_TO_SOT_SMD:TDSON-8-1, B.Cu at (132.9, 119.2)
- added Q4: BSC061N08NS5, Package_TO_SOT_SMD:TDSON-8-1, B.Cu at (116.4, 112.5)
- added Q5: BSC061N08NS5, Package_TO_SOT_SMD:TDSON-8-1, B.Cu at (132.9, 112.5)
- added Q6: BSC061N08NS5, Package_TO_SOT_SMD:TDSON-8-1, B.Cu at (124.7, 119.2)
- added R1: 200k, Resistor_SMD:R_0603_1608Metric_Pad0.98x0.95mm_HandSolder, F.Cu at (147.0, 81.3)
- added R10: 22k, Resistor_SMD:R_0603_1608Metric_Pad0.98x0.95mm_HandSolder, F.Cu at (175.0, 94.5)
- added R2: 10, Resistor_SMD:R_0603_1608Metric_Pad0.98x0.95mm_HandSolder, F.Cu at (147.0, 83.8)
- added R3: 22k, Resistor_SMD:R_0603_1608Metric_Pad0.98x0.95mm_HandSolder, F.Cu at (111.3, 87.4)
- added R4: 22k, Resistor_SMD:R_0603_1608Metric_Pad0.98x0.95mm_HandSolder, F.Cu at (115.6, 87.4)
- added R5: 22k, Resistor_SMD:R_0603_1608Metric_Pad0.98x0.95mm_HandSolder, F.Cu at (111.3, 89.9)
- added R6: 200k, Resistor_SMD:R_0603_1608Metric_Pad0.98x0.95mm_HandSolder, F.Cu at (179.3, 89.4)
- added R7: 10, Resistor_SMD:R_0603_1608Metric_Pad0.98x0.95mm_HandSolder, F.Cu at (183.7, 89.4)
- added R8: 22k, Resistor_SMD:R_0603_1608Metric_Pad0.98x0.95mm_HandSolder, F.Cu at (175.0, 91.9)
- added R9: 22k, Resistor_SMD:R_0603_1608Metric_Pad0.98x0.95mm_HandSolder, F.Cu at (175.0, 89.4)
- added U1: STM32F334R8Tx, Package_QFP:LQFP-64_10x10mm_P0.5mm, F.Cu at (152.4, 101.6)
- added U2: DRV8301DCAR, Package_SO:HTSSOP-56-1EP_6.1x14mm_P0.5mm_EP3.61x6.35mm, F.Cu at (169.7, 81.2)
- added U3: DRV8301DCAR, Package_SO:HTSSOP-56-1EP_6.1x14mm_P0.5mm_EP3.61x6.35mm, F.Cu at (135.1, 81.3)
Routing:
- added copper zone on B.Cu, net GND
- added copper zone on F.Cu, net GND
Other:
- board outline added: 100 x 80 mm
- copper layers 0 -> 2
