File: FOC.kicad_sch (KiCad schematic)
At the start: 0 parts

Commit message: 123
Parts:
- added C1: 100u, Capacitor_Tantalum_SMD:CP_EIA-7343-30_AVX-N_Pad2.25x2.55mm_HandSolder, symbol Device:C_Polarized_Small
- added C10, C11, C12, C13, C14, C21, C23, C3, C5, C7, C9: 100n, Capacitor_SMD:C_0603_1608Metric_Pad1.08x0.95mm_HandSolder, symbol Device:C_Small
- added C15, C19: 22n, Capacitor_SMD:C_0603_1608Metric_Pad1.08x0.95mm_HandSolder, symbol Device:C_Small
- added C16, C24: 2.2u, Capacitor_SMD:C_0603_1608Metric_Pad1.08x0.95mm_HandSolder, symbol Device:C_Small
- added C17, C18, C25, C26: 1u, Capacitor_SMD:C_0603_1608Metric_Pad1.08x0.95mm_HandSolder, symbol Device:C_Small
- added C2, C27: 15n, Capacitor_SMD:C_0603_1608Metric_Pad1.08x0.95mm_HandSolder, symbol Device:C_Small
- added C20, C22, C6, C8: 4.7u, Capacitor_SMD:C_0603_1608Metric_Pad1.08x0.95mm_HandSolder, symbol Device:C_Small
- added C4: 47u, Capacitor_Tantalum_SMD:CP_EIA-7343-30_AVX-N_Pad2.25x2.55mm_HandSolder, symbol Device:C_Polarized_Small
- added D1: D_S, Diode_SMD:D_SOD-323_HandSoldering, symbol Device:D_Schottky_Small_Filled
- added J1: PWR, Connector_AMASS:AMASS_XT60-M_1x02_P7.20mm_Vertical, symbol Connector_Generic:Conn_01x02
- added L1: 22u, Inductor_SMD:L_Sumida_CDMC6D28_7.25x6.5mm, symbol Device:L_Small
- added Q?: BSC265N10LSFG, Package_TO_SOT_SMD:TDSON-8-1, symbol Transistor_FET:BSC265N10LSFG
- added R1, R6: 200k, Resistor_SMD:R_0603_1608Metric_Pad0.98x0.95mm_HandSolder, symbol Device:R_Small
- added R10, R3, R4, R5, R8, R9: 22k, Resistor_SMD:R_0603_1608Metric_Pad0.98x0.95mm_HandSolder, symbol Device:R_Small
- added R2, R7: 10, Resistor_SMD:R_0603_1608Metric_Pad0.98x0.95mm_HandSolder, symbol Device:R_Small
- added U1: STM32F334R8Tx, Package_QFP:LQFP-64_10x10mm_P0.5mm, symbol MCU_ST_STM32F3:STM32F334R8Tx
- added U2, U3: DRV8301DCAR, Package_SO:HTSSOP-56-1EP_6.1x14mm_P0.5mm_EP3.61x6.35mm, symbol DRV8301DCAR:DRV8301DCAR
Connections:
- new net: C19.1, U2.14 (CP1)
- new net: C19.2, U2.15 (CP2)
- new net: R3.1, U3.4 (PWRGD)
- new net: R1.2, U3.1 (RT_CLK)
- new net: R9.1, U2.6 (~FAULT)
- new net: C16.2, U3.13 (GVDD)
- new net: C25.2, U2.27 (AVDD)
- new net: R8.1, U2.4 (PWRGD)
- new net: R2.2, U3.7 (DTC)
- new net: C18.2, U3.23 (DVDD)
- new net: R6.2, U2.1 (RT_CLK)
- new net: R5.1, U3.5 (~OCTW)
- new net: C3.2, U3.52 (BST_BK)
- new net: R10.1, U2.5 (~OCTW)
- new net: C26.2, U2.23 (DVDD)
- new net: D1.1 (K), L1.1, U3.50 (PH), U3.51 (PH)
- new net: C2.2, U3.56 (SS_TR)
- new net: C15.1, U3.14 (CP1)
- new net: C15.2, U3.15 (CP2)
- new net: Q?.1 (S), Q?.2 (S), Q?.3 (S)
- new net: C17.2, U3.27 (AVDD)
- new net: R4.1, U3.6 (~FAULT)
- new net: C24.2, U2.13 (GVDD)
- new net: U2.50 (PH), U2.51 (PH)
- new net: C27.2, U2.56 (SS_TR)
- new net: R7.2, U2.7 (DTC)
- new net +3V3: C10.2, C11.2, C12.2, C13.2, C14.2, C3.1, C4.1, C5.2, L1.2, R10.2, R3.2, R4.2, R5.2, R8.2, R9.2, U1.13 (VDDA), U1.19 (VDD), U1.32 (VDD), U1.48 (VDD), U1.64 (VDD), U2.49 (VDD_SPI), U3.49 (VDD_SPI)
- new net COMP: U3.2 (COMP)
- new net CS0: U3.8 (~SCS)
- new net GND: C1.2, C10.1, C11.1, C12.1, C13.1, C14.1, C16.1, C17.1, C18.1, C2.1, C20.1, C21.1, C22.1, C23.1, C24.1, C25.1, C26.1, C27.1, C4.2, C5.1, C6.1, C7.1, C8.1, C9.1, D1.2 (A), J1.2 (Pin_2), R1.1, R2.1, R6.1, R7.1, U1.12 (VSSA), U1.18 (VSS), U1.31 (VSS), U1.47 (VSS), U1.63 (VSS), U2.28 (AGND), U2.57 (GND), U3.28 (AGND), U3.57 (GND)
- new net MISO: U2.10 (SDO), U3.10 (SDO)
- new net MOSI: U2.9 (SDI), U3.9 (SDI)
- new net SCLK: U2.11 (SCLK), U3.11 (SCLK)
- new net SENSE_REF: U3.24 (REF)
- new net VDD: C1.1, C20.2, C21.2, C22.2, C23.2, C6.2, C7.2, C8.2, C9.2, J1.1 (Pin_1), U2.29 (PVDD1), U2.53 (PVDD2), U2.54 (PVDD2), U3.29 (PVDD1), U3.53 (PVDD2), U3.54 (PVDD2)
